File: FRONT/MIDI_DIN_front.sch (KiCad schematic (older format))
At the start: 6 parts, among them J1 Screw_Terminal_01x01, J2 Screw_Terminal_01x01, J3 Screw_Terminal_01x01, J4 Screw_Terminal_01x01

Commit message: Add custom symbols and footprints
Parts:
- H1, H2: footprint CustomLib:DIN_Hole_Hirschmann -> Custom_FP:DIN_Hole_Hirschmann
- J1, J2, J3, J4: footprint CustomLib:Wide_M3 -> Custom_FP:Wide_M3
Changed lines of the file:
@@
 F 0 "H1" H 3400 2546 50  0000 L CNN
 F 1 "DIN_IN" H 3400 2455 50  0000 L CNN
-F 2 "CustomLib:DIN_Hole_Hirschmann" H 3300 2500 50  0001 C CNN
+F 2 "Custom_FP:DIN_Hole_Hirschmann" H 3300 2500 50  0001 C CNN
 F 3 "~" H 3300 2500 50  0001 C CNN
 	1    3300 2500
@@
 F 0 "H2" H 4550 2546 50  0000 L CNN
 F 1 "DIN_OUT" H 4550 2455 50  0000 L CNN
-F 2 "CustomLib:DIN_Hole_Hirschmann" H 4450 2500 50  0001 C CNN
+F 2 "Custom_FP:DIN_Hole_Hirschmann" H 4450 2500 50  0001 C CNN
 F 3 "~" H 4450 2500 50  0001 C CNN
 	1    4450 2500
@@
 F 0 "J1" H 3330 3192 50  0000 L CNN
 F 1 "Screw_Terminal_01x01" H 3330 3101 50  0000 L CNN
-F 2 "CustomLib:Wide_M3" H 3250 3150 50  0001 C CNN
+F 2 "Custom_FP:Wide_M3" H 3250 3150 50  0001 C CNN
 F 3 "~" H 3250 3150 50  0001 C CNN
 	1    3250 3150
@@
 F 0 "J2" H 3330 3392 50  0000 L CNN
 F 1 "Screw_Terminal_01x01" H 3330 3301 50  0000 L CNN
-F 2 "CustomLib:Wide_M3" H 3250 3350 50  0001 C CNN
+F 2 "Custom_FP:Wide_M3" H 3250 3350 50  0001 C CNN
 F 3 "~" H 3250 3350 50  0001 C CNN
 	1    3250 3350
@@
 F 0 "J3" H 3330 3592 50  0000 L CNN
 F 1 "Screw_Terminal_01x01" H 3330 3501 50  0000 L CNN
-F 2 "CustomLib:Wide_M3" H 3250 3550 50  0001 C CNN
+F 2 "Custom_FP:Wide_M3" H 3250 3550 50  0001 C CNN
 F 3 "~" H 3250 3550 50  0001 C CNN
 	1    3250 3550
@@
 F 0 "J4" H 3330 3792 50  0000 L CNN
 F 1 "Screw_Terminal_01x01" H 3330 3701 50  0000 L CNN
-F 2 "CustomLib:Wide_M3" H 3250 3750 50  0001 C CNN
+F 2 "Custom_FP:Wide_M3" H 3250 3750 50  0001 C CNN
 F 3 "~" H 3250 3750 50  0001 C CNN
 	1    3250 3750
