File: FRONT/MIDI_DIN_front.kicad_pcb (KiCad board)
At the start: 2 copper layers, 30 x 128.5 mm, 6 parts, among them J1 Screw_Terminal_01x01, J2 Screw_Terminal_01x01, J3 Screw_Terminal_01x01, J4 Screw_Terminal_01x01

Commit message: Update module name
Other:
- board text added: "2"
- board text added: "M IDI DIN"
- board text removed: "MIDIBUS DIN"
Changed lines of the file:
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@@
-(kicad_pcb (version 20171130) (host pcbnew "(5.1.6)-1")
+(kicad_pcb (version 20171130) (host pcbnew "(5.1.10)-1")
   (general
     (thickness 1.6)
-    (drawings 38)
+    (drawings 39)
     (tracks 0)
     (zones 0)
@@
       (effects (font (size 1 1) (thickness 0.15)))
     )
+    (fp_circle (center 0 0) (end 10 0) (layer F.Fab) (width 0.12))
+    (fp_line (start -1.5 -10) (end -1.499999 -8.95) (layer Dwgs.User) (width 0.12))
+    (fp_line (start 1.5 -10) (end -1.5 -10) (layer Dwgs.User) (width 0.12))
+    (fp_line (start 1.479934 -8.95334) (end 1.5 -10) (layer Dwgs.User) (width 0.12))
+    (fp_poly (pts (xy 7 12.25) (xy 4.5 14.25) (xy -4.5 14.25) (xy -7 12.25)
+      (xy -7 10.25) (xy 7 10.25)) (layer B.Mask) (width 0.1))
+    (fp_poly (pts (xy 7 12.25) (xy 4.5 14.25) (xy -4.5 14.25) (xy -7 12.25)
+      (xy -7 10.25) (xy 7 10.25)) (layer F.Mask) (width 0.1))
+    (fp_line (start 0 9) (end 0 10.25) (layer Dwgs.User) (width 0.12))
+    (fp_line (start 0.25 10.25) (end -0.25 10.25) (layer Dwgs.User) (width 0.12))
+    (fp_line (start 0 10.25) (end 0 14.25) (layer Dwgs.User) (width 0.12))
     (fp_line (start -0.25 14.25) (end 0.25 14.25) (layer Dwgs.User) (width 0.12))
-    (fp_line (start 0 10.25) (end 0 14.25) (layer Dwgs.User) (width 0.12))
-    (fp_line (start 0.25 10.25) (end -0.25 10.25) (layer Dwgs.User) (width 0.12))
-    (fp_line (start 0 9) (end 0 10.25) (layer Dwgs.User) (width 0.12))
-    (fp_poly (pts (xy 7 12.25) (xy 4.5 14.25) (xy -4.5 14.25) (xy -7 12.25)
-      (xy -7 10.25) (xy 7 10.25)) (layer F.Mask) (width 0.1))
-    (fp_poly (pts (xy 7 12.25) (xy 4.5 14.25) (xy -4.5 14.25) (xy -7 12.25)
-      (xy -7 10.25) (xy 7 10.25)) (layer B.Mask) (width 0.1))
-    (fp_line (start 1.479934 -8.95334) (end 1.5 -10) (layer Dwgs.User) (width 0.12))
-    (fp_line (start 1.5 -10) (end -1.5 -10) (layer Dwgs.User) (width 0.12))
-    (fp_line (start -1.5 -10) (end -1.499999 -8.95) (layer Dwgs.User) (width 0.12))
-    (fp_circle (center 0 0) (end 10 0) (layer F.Fab) (width 0.12))
     (fp_arc (start 0 0) (end -1.499999 -8.95) (angle -341.1) (layer Dwgs.User) (width 0.12))
   )
@@
       (effects (font (size 1 1) (thickness 0.15)))
     )
+    (fp_circle (center 0 0) (end 10 0) (layer F.Fab) (width 0.12))
+    (fp_line (start -1.5 -10) (end -1.499999 -8.95) (layer Dwgs.User) (width 0.12))
+    (fp_line (start 1.5 -10) (end -1.5 -10) (layer Dwgs.User) (width 0.12))
+    (fp_line (start 1.479934 -8.95334) (end 1.5 -10) (layer Dwgs.User) (width 0.12))
+    (fp_poly (pts (xy 7 12.25) (xy 4.5 14.25) (xy -4.5 14.25) (xy -7 12.25)
+      (xy -7 10.25) (xy 7 10.25)) (layer B.Mask) (width 0.1))
+    (fp_poly (pts (xy 7 12.25) (xy 4.5 14.25) (xy -4.5 14.25) (xy -7 12.25)
+      (xy -7 10.25) (xy 7 10.25)) (layer F.Mask) (width 0.1))
+    (fp_line (start 0 9) (end 0 10.25) (layer Dwgs.User) (width 0.12))
+    (fp_line (start 0.25 10.25) (end -0.25 10.25) (layer Dwgs.User) (width 0.12))
+    (fp_line (start 0 10.25) (end 0 14.25) (layer Dwgs.User) (width 0.12))
     (fp_line (start -0.25 14.25) (end 0.25 14.25) (layer Dwgs.User) (width 0.12))
-    (fp_line (start 0 10.25) (end 0 14.25) (layer Dwgs.User) (width 0.12))
-    (fp_line (start 0.25 10.25) (end -0.25 10.25) (layer Dwgs.User) (width 0.12))
-    (fp_line (start 0 9) (end 0 10.25) (layer Dwgs.User) (width 0.12))
-    (fp_poly (pts (xy 7 12.25) (xy 4.5 14.25) (xy -4.5 14.25) (xy -7 12.25)
-      (xy -7 10.25) (xy 7 10.25)) (layer F.Mask) (width 0.1))
-    (fp_poly (pts (xy 7 12.25) (xy 4.5 14.25) (xy -4.5 14.25) (xy -7 12.25)
-      (xy -7 10.25) (xy 7 10.25)) (layer B.Mask) (width 0.1))
-    (fp_line (start 1.479934 -8.95334) (end 1.5 -10) (layer Dwgs.User) (width 0.12))
-    (fp_line (start 1.5 -10) (end -1.5 -10) (layer Dwgs.User) (width 0.12))
-    (fp_line (start -1.5 -10) (end -1.499999 -8.95) (layer Dwgs.User) (width 0.12))
-    (fp_circle (center 0 0) (end 10 0) (layer F.Fab) (width 0.12))
     (fp_arc (start 0 0) (end -1.499999 -8.95) (angle -341.1) (layer Dwgs.User) (width 0.12))
+  )
+  (gr_text 2 (at 89.25 46.25) (layer F.Mask)
+    (effects (font (size 1.7 1.7) (thickness 0.25)))
   )
   (gr_arc (start 92.5 119.35) (end 93.5 119.35) (angle -90) (layer Edge.Cuts) (width 0.05))
@@
   (gr_line (start 90 120.6) (end 90 125.5) (layer Dwgs.User) (width 0.15))
   (gr_line (start 73.25 53) (end 105.75 53) (layer F.Mask) (width 0.4))
-  (gr_text "MIDIBUS\nDIN" (at 90 49.25) (layer F.Mask)
+  (gr_text "M IDI\nDIN" (at 90 49.25) (layer F.Mask)
     (effects (font (size 2 2) (thickness 0.25)))
   )

Commit message: Update front panel
Connections:
- J1 pad 1: GND -> unconnected-(J1-Pin_1-Pad1)
- J2 pad 1: GND -> unconnected-(J2-Pin_1-Pad1)
- J3 pad 1: GND -> unconnected-(J3-Pin_1-Pad1)
- J4 pad 1: GND -> unconnected-(J4-Pin_1-Pad1)
Routing:
- added copper zone on B.Cu, net unconnected-(J2-Pin_1-Pad1)
- added copper zone on F.Cu, net unconnected-(J2-Pin_1-Pad1)
- removed copper zone on B.Cu, net GND
- removed copper zone on F.Cu, net GND
Other:
- net class Default removed

Commit message: Finalize module
Parts:
- moved H1 5.02 mm to (85.0, 90.0)
- moved H2 5.02 mm to (85.0, 136.0)
- moved J1 5.02 mm to (92.5, 166.0)
- moved J2 5.02 mm to (92.5, 43.5)
- moved J3 5.02 mm to (77.5, 166.0)
- moved J4 5.02 mm to (77.5, 43.5)
Connections:
- J1 pad 1: unconnected-(J1-Pin_1-Pad1) -> Net-(J1-Pin_1)
- J2 pad 1: unconnected-(J2-Pin_1-Pad1) -> Net-(J1-Pin_1)
- J3 pad 1: unconnected-(J3-Pin_1-Pad1) -> Net-(J1-Pin_1)
- J4 pad 1: unconnected-(J4-Pin_1-Pad1) -> Net-(J1-Pin_1)
Routing:
- added copper zone on B.Cu, net Net-(J1-Pin_1)
- added copper zone on F.Cu, net Net-(J1-Pin_1)
- removed copper zone on B.Cu, net unconnected-(J2-Pin_1-Pad1)
- removed copper zone on F.Cu, net unconnected-(J2-Pin_1-Pad1)
Other:
- rule pad_to_mask_clearance: 0.05 -> 0
