File: FRONT/MIDI_DIN_front.kicad_sch (KiCad schematic)
At the start: 6 parts, among them J1 Screw_Terminal_01x01, J2 Screw_Terminal_01x01, J3 Screw_Terminal_01x01, J4 Screw_Terminal_01x01

Commit message: Finalize module
Connections:
- net at J1.1 (Pin_1): now also J2.1 (Pin_1), J3.1 (Pin_1), J4.1 (Pin_1)
- no-connect marks 4 -> 0
Changed lines of the file:
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@@
 (kicad_sch (version 20230121) (generator eeschema)
   (paper "A4")
-  (no_connect (at 77.47 80.01))
-  (no_connect (at 77.47 90.17))
-  (no_connect (at 77.47 95.25))
-  (no_connect (at 77.47 85.09))
+  (junction (at 73.025 85.09) (diameter 0) (color 0 0 0 0)
+  )
+  (junction (at 73.025 90.17) (diameter 0) (color 0 0 0 0)
+  )
+  (wire (pts (xy 73.025 95.25) (xy 77.47 95.25))
+    (stroke (width 0) (type default))
+  )
+  (wire (pts (xy 73.025 85.09) (xy 73.025 90.17))
+    (stroke (width 0) (type default))
+  )
+  (wire (pts (xy 73.025 90.17) (xy 77.47 90.17))
+    (stroke (width 0) (type default))
+  )
+  (wire (pts (xy 77.47 80.01) (xy 73.025 80.01))
+    (stroke (width 0) (type default))
+  )
+  (wire (pts (xy 73.025 90.17) (xy 73.025 95.25))
+    (stroke (width 0) (type default))
+  )
+  (wire (pts (xy 73.025 80.01) (xy 73.025 85.09))
+    (stroke (width 0) (type default))
+  )
+  (wire (pts (xy 73.025 85.09) (xy 77.47 85.09))
+    (stroke (width 0) (type default))
+  )
   (symbol (lib_id "Mechanical:MountingHole") (at 83.82 63.5 0) (unit 1)
     (in_bom yes) (on_board yes) (dnp no)
