File: CORE/MIDI_DIN.sch (KiCad schematic (older format))
At the start: 56 parts, among them J1 Conn_02x08_Odd_Even, J2 USB_C_Receptacle_USB2.0, J3 Conn_01x04, J5 DIN-5_180degree, J6 DIN-5_180degree, J7 Conn_01x06, Q1 MMBT3904, SW1 SW_SPDT, SW2 SW_Push_DPDT, U1 ATSAMD21G15B-A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

Commit message: Update termination values
Parts:
- C16: value 22nF -> 4.7nF
- J2: symbol MIDI_DIN-rescue:USB_C_Receptacle_USB2.0-Connector -> Connector:USB_C_Receptacle_USB2.0
- R18, R19: value 120 -> 56
Changed lines of the file:
@@
 $EndComp
 $Comp
-L MIDI_DIN-rescue:USB_C_Receptacle_USB2.0-Connector J2
+L Connector:USB_C_Receptacle_USB2.0 J2
 U 1 1 60B5F154
 P 1200 6000
@@
 P 10550 3250
 F 0 "R18" H 10620 3296 50  0000 L CNN
-F 1 "120" H 10620 3205 50  0000 L CNN
+F 1 "56" H 10620 3205 50  0000 L CNN
 F 2 "Resistor_SMD:R_0603_1608Metric" V 10480 3250 50  0001 C CNN
 F 3 "~" H 10550 3250 50  0001 C CNN
@@
 P 10550 3650
 F 0 "R19" H 10620 3696 50  0000 L CNN
-F 1 "120" H 10620 3605 50  0000 L CNN
+F 1 "56" H 10620 3605 50  0000 L CNN
 F 2 "Resistor_SMD:R_0603_1608Metric" V 10480 3650 50  0001 C CNN
 F 3 "~" H 10550 3650 50  0001 C CNN
@@
 P 10900 3500
 F 0 "C16" H 11015 3546 50  0000 L CNN
-F 1 "22nF" H 11015 3455 50  0000 L CNN
+F 1 "4.7nF" H 11015 3455 50  0000 L CNN
 F 2 "Capacitor_SMD:C_0603_1608Metric" H 10938 3350 50  0001 C CNN
 F 3 "~" H 10900 3500 50  0001 C CNN

Commit message: Add custom symbols and footprints
Parts:
- J1: footprint CustomLib:Header_2x8_Shrouded_SMD -> Custom_FP:Header_2x8_Shrouded_SMD
- J2: footprint CustomLib:USB_C_Receptacle_GCT_USB4085_Slimmed -> Custom_FP:USB_C_Receptacle_GCT_USB4085_Slimmed
- J3: footprint CustomLib:MicroMatch_04_Vertical_SMD -> Custom_FP:MicroMatch_04_Vertical_SMD
- J5, J6: value DIN-5_180degree -> MAB5100S; footprint CustomLib:DIN-5_Hirschmann -> Custom_FP:DIN-5_Hirschmann_MAB5100S
- SW1: footprint CustomLib:SlideSwitch-SS12D10 -> Custom_FP:SlideSwitch-SS12D10
- SW2: footprint CustomLib:SlideDPDT_JS202011 -> Custom_FP:SlideDPDT_JS202011
- Y1: footprint CustomLib:Crystal_2pin_2.0x2.5mm -> Custom_FP:Crystal_2pin_2.0x2.5mm
Changed lines of the file:
@@
 P 10250 1600
 F 0 "J5" V 10204 1370 50  0000 R CNN
-F 1 "DIN-5_180degree" V 10295 1370 50  0000 R CNN
-F 2 "CustomLib:DIN-5_Hirschmann" H 10250 1600 50  0001 C CNN
+F 1 "MAB5100S" V 10295 1370 50  0000 R CNN
+F 2 "Custom_FP:DIN-5_Hirschmann_MAB5100S" H 10250 1600 50  0001 C CNN
 F 3 "http://www.mouser.com/ds/2/18/40_c091_abd_e-75918.pdf" H 10250 1600 50  0001 C CNN
 	1    10250 1600
@@
 P 8400 3100
 F 0 "J6" V 8354 2870 50  0000 R CNN
-F 1 "DIN-5_180degree" V 8445 2870 50  0000 R CNN
-F 2 "CustomLib:DIN-5_Hirschmann" H 8400 3100 50  0001 C CNN
+F 1 "MAB5100S" V 8445 2870 50  0000 R CNN
+F 2 "Custom_FP:DIN-5_Hirschmann_MAB5100S" H 8400 3100 50  0001 C CNN
 F 3 "http://www.mouser.com/ds/2/18/40_c091_abd_e-75918.pdf" H 8400 3100 50  0001 C CNN
 	1    8400 3100
@@
 F 0 "SW1" H 6650 1685 50  0000 C CNN
 F 1 "SW_SPDT" H 6650 1594 50  0000 C CNN
-F 2 "CustomLib:SlideSwitch-SS12D10" H 6650 1400 50  0001 C CNN
+F 2 "Custom_FP:SlideSwitch-SS12D10" H 6650 1400 50  0001 C CNN
 F 3 "~" H 6650 1400 50  0001 C CNN
 	1    6650 1400
@@
 F 0 "J1" H 3600 7717 50  0000 C CNN
 F 1 "Conn_02x08_Odd_Even" H 3600 7626 50  0000 C CNN
-F 2 "CustomLib:Header_2x8_Shrouded_SMD" H 3550 7200 50  0001 C CNN
+F 2 "Custom_FP:Header_2x8_Shrouded_SMD" H 3550 7200 50  0001 C CNN
 F 3 "~" H 3550 7200 50  0001 C CNN
 	1    3550 7200
@@
 F 0 "J2" H 1307 6867 50  0000 C CNN
 F 1 "USB_C_Receptacle_USB2.0" H 1307 6776 50  0000 C CNN
-F 2 "CustomLib:USB_C_Receptacle_GCT_USB4085_Slimmed" H 1350 6000 50  0001 C CNN
+F 2 "Custom_FP:USB_C_Receptacle_GCT_USB4085_Slimmed" H 1350 6000 50  0001 C CNN
 F 3 "https://www.usb.org/sites/default/files/documents/usb_type-c.zip" H 1350 6000 50  0001 C CNN
 	1    1200 6000
@@
 F 0 "SW2" H 10150 4035 50  0000 C CNN
 F 1 "SW_Push_DPDT" H 10150 3944 50  0000 C CNN
-F 2 "CustomLib:SlideDPDT_JS202011" H 10150 3750 50  0001 C CNN
+F 2 "Custom_FP:SlideDPDT_JS202011" H 10150 3750 50  0001 C CNN
 F 3 "~" H 10150 3750 50  0001 C CNN
 	1    10150 3550
@@
 F 0 "J3" H 10530 5142 50  0000 L CNN
 F 1 "Conn_01x04" H 10530 5051 50  0000 L CNN
-F 2 "CustomLib:MicroMatch_04_Vertical_SMD" H 10450 5150 50  0001 C CNN
+F 2 "Custom_FP:MicroMatch_04_Vertical_SMD" H 10450 5150 50  0001 C CNN
 F 3 "~" H 10450 5150 50  0001 C CNN
 	1    10450 5150
@@
 F 0 "Y1" V 5854 6031 50  0000 L CNN
 F 1 "20MHz" V 5945 6031 50  0000 L CNN
-F 2 "CustomLib:Crystal_2pin_2.0x2.5mm" H 5900 5900 50  0001 C CNN
+F 2 "Custom_FP:Crystal_2pin_2.0x2.5mm" H 5900 5900 50  0001 C CNN
 F 3 "~" H 5900 5900 50  0001 C CNN
 	1    5900 5900

Commit message: Update PCB
Fixed stuff
Parts:
- removed Q1: MMBT3904, Package_TO_SOT_SMD:SOT-23, symbol Transistor_BJT:MMBT3904
- added Q1: MMBT3906, Package_TO_SOT_SMD:SOT-23, symbol Transistor_BJT:MMBT3906
- added R17: 10k, Resistor_SMD:R_0603_1608Metric, symbol Device:R
- added SW3: PROG, Custom_FP:Tactile_angled_5x5.4_SMD, symbol Switch:SW_SPST
- added SW4: SW_DIP_x04, Button_Switch_SMD:SW_DIP_SPSTx04_Slide_Copal_CHS-04B_W7.62mm_P1.27mm, symbol Switch:SW_DIP_x04
- added SW5: RST, Custom_FP:Tactile_angled_5x5.4_SMD, symbol Switch:SW_SPST
- J2: footprint Custom_FP:USB_C_Receptacle_GCT_USB4085_Slimmed -> Connector_USB:USB_C_Receptacle_HRO_TYPE-C-31-M-12
Connections:
- net +3V3: now also Q1.2 (E), R17.1; no longer R9.1
- net GND: now also R10.2, SW3.2 (B), SW4.1, SW4.2, SW4.3, SW4.4, SW5.2 (B)
- net RST: now also SW5.1 (A)
- net at R7.1: now also Q1.1 (B)
- net at U1.19 (PB10): now also SW4.6
- net at U1.20 (PB11): now also SW4.5
- net PROG: now reaches U1.41 (PA28)
- net PROG: now also R17.2, SW3.1 (A)
- net at U1.7 (PB08): now also SW4.8
- net at U1.8 (PB09): now also SW4.7
- new net: Q1.3 (C), R9.1
Other:
- moved on the sheet: J6, R10, R15, R7, R9

Commit message: Add horizontal prog header
Parts:
- J7: footprint Connector_PinHeader_2.54mm:PinHeader_2x03_P2.54mm_Vertical_SMD -> Custom_FP:TSM103-DH
Changed lines of the file:
@@
 encoding utf-8
 Sheet 1 1
-Title ""
+Title "MIDIBUS - DIN"
 Date ""
-Rev ""
+Rev "2.1"
 Comp ""
 Comment1 ""
@@
 F 0 "J7" H 1430 4292 50  0000 L CNN
 F 1 "Conn_01x06" H 1430 4201 50  0000 L CNN
-F 2 "Connector_PinHeader_2.54mm:PinHeader_2x03_P2.54mm_Vertical_SMD" H 1350 4300 50  0001 C CNN
+F 2 "Custom_FP:TSM103-DH" H 1350 4300 50  0001 C CNN
 F 3 "~" H 1350 4300 50  0001 C CNN
 	1    1350 4300

Commit message: Minor adjustments
Parts:
- R18, R19: value 56 -> 62
Other:
- moved on the sheet: C16
Changed lines of the file:
@@
 P 10550 3250
 F 0 "R18" H 10620 3296 50  0000 L CNN
-F 1 "56" H 10620 3205 50  0000 L CNN
+F 1 "62" H 10620 3205 50  0000 L CNN
 F 2 "Resistor_SMD:R_0603_1608Metric" V 10480 3250 50  0001 C CNN
 F 3 "~" H 10550 3250 50  0001 C CNN
@@
 P 10550 3650
 F 0 "R19" H 10620 3696 50  0000 L CNN
-F 1 "56" H 10620 3605 50  0000 L CNN
+F 1 "62" H 10620 3605 50  0000 L CNN
 F 2 "Resistor_SMD:R_0603_1608Metric" V 10480 3650 50  0001 C CNN
 F 3 "~" H 10550 3650 50  0001 C CNN
@@
 L power:GND #PWR0105
 U 1 1 60F03FCF
-P 10900 3700
-F 0 "#PWR0105" H 10900 3450 50  0001 C CNN
-F 1 "GND" H 10905 3527 50  0000 C CNN
-F 2 "" H 10900 3700 50  0001 C CNN
-F 3 "" H 10900 3700 50  0001 C CNN
-	1    10900 3700
-	1    0    0    -1
-$EndComp
-Wire Wire Line
-	10900 3700 10900 3650
+P 10750 4200
+F 0 "#PWR0105" H 10750 3950 50  0001 C CNN
+F 1 "GND" H 10755 4027 50  0000 C CNN
+F 2 "" H 10750 4200 50  0001 C CNN
+F 3 "" H 10750 4200 50  0001 C CNN
+	1    10750 4200
+	1    0    0    -1
+$EndComp
+Wire Wire Line
+	10750 4200 10750 4150
 Text GLabel 10300 4850 2    50   BiDi ~ 0
 MIDIBUS+
@@
 $EndComp
 Wire Wire Line
-	9150 6300 9150 6250
-Wire Wire Line
 	9950 3750 9850 3750
 Wire Wire Line
@@
 Wire Wire Line
 	6900 6200 6900 6100
-$Comp
-L Device:C C10
-U 1 1 610A595F
-P 8000 5950
-F 0 "C10" H 8115 5996 50  0000 L CNN
-F 1 "100nF" H 8115 5905 50  0000 L CNN
-F 2 "Capacitor_SMD:C_0603_1608Metric" H 8038 5800 50  0001 C CNN
-F 3 "~" H 8000 5950 50  0001 C CNN
-	1    8000 5950
-	0    1    1    0
-$EndComp
 Wire Wire Line
 	8200 5950 8150 5950
-Wire Wire Line
-	7800 5950 7850 5950
-$Comp
-L power:GND #PWR0136
-U 1 1 610CB3DD
-P 7800 5950
-F 0 "#PWR0136" H 7800 5700 50  0001 C CNN
-F 1 "GND" H 7805 5777 50  0000 C CNN
-F 2 "" H 7800 5950 50  0001 C CNN
-F 3 "" H 7800 5950 50  0001 C CNN
-	1    7800 5950
-	0    1    1    0
-$EndComp
 Wire Wire Line
 	4050 7000 4750 7000
@@
 Connection ~ 9750 5250
 Wire Wire Line
-	9750 5250 9750 5750
-Wire Wire Line
 	10150 5350 10150 5500
 Connection ~ 10150 5350
@@
 L Device:C C16
 U 1 1 60E87FD8
-P 10900 3500
-F 0 "C16" H 11015 3546 50  0000 L CNN
-F 1 "4.7nF" H 11015 3455 50  0000 L CNN
-F 2 "Capacitor_SMD:C_0603_1608Metric" H 10938 3350 50  0001 C CNN
-F 3 "~" H 10900 3500 50  0001 C CNN
-	1    10900 3500
+P 10750 4000
+F 0 "C16" H 10865 4046 50  0000 L CNN
+F 1 "4.7nF" H 10865 3955 50  0000 L CNN
+F 2 "Capacitor_SMD:C_0603_1608Metric" H 10788 3850 50  0001 C CNN
+F 3 "~" H 10750 4000 50  0001 C CNN
+	1    10750 4000
 	1    0    0    -1
 $EndComp
@@
 U 1 1 60F2A7B0
 P 6900 5600
-F 0 "U4" H 6900 6281 50  0000 C CNN
-F 1 "MCP2517FD-xSL" H 6900 6190 50  0000 C CNN
+F 0 "U4" H 7200 6150 50  0000 C CNN
+F 1 "MCP2517FD-xSL" H 7250 6050 50  0000 C CNN
 F 2 "Package_SO:SOIC-14_3.9x8.7mm_P1.27mm" H 6900 4600 50  0001 C CNN
 F 3 "https://ww1.microchip.com/downloads/en/DeviceDoc/20005688A.pdf" H 6900 5850 50  0001 C CNN
@@
 	1    0    0    -1
 $EndComp
-$Comp
-L Interface_CAN_LIN:MCP2558FD-xMF U5
-U 1 1 60F56096
-P 9150 5850
-F 0 "U5" H 9150 6431 50  0000 C CNN
-F 1 "TLE9250V" H 9150 6340 50  0000 C CNN
-F 2 "Package_SO:Infineon_PG-DSO-8-27_3.9x4.9mm_EP2.65x3mm" H 9150 5250 50  0001 C CNN
-F 3 "https://ww1.microchip.com/downloads/en/DeviceDoc/20005533A.pdf" H 9150 5850 50  0001 C CNN
-	1    9150 5850
-	1    0    0    -1
-$EndComp
 Wire Wire Line
 	10350 3650 10400 3650
@@
 Wire Wire Line
 	10750 3650 10700 3650
-Wire Wire Line
-	10750 3250 10900 3250
-Wire Wire Line
-	10900 3250 10900 3350
-Connection ~ 10750 3250
-Wire Wire Line
-	9650 5950 9850 5950
-Wire Wire Line
-	9850 5150 9850 5950
-Wire Wire Line
-	9650 5750 9750 5750
 Wire Wire Line
 	9150 4900 9150 4950
@@
 	8600 4950 9150 4950
 Connection ~ 9150 4950
-Wire Wire Line
-	9150 4950 9150 5450
 $Comp
 L power:GND #PWR05
@@
 	1    0    0    -1
 $EndComp
-$Comp
-L power:+3V3 #PWR04
-U 1 1 610BDED3
-P 8200 5900
-F 0 "#PWR04" H 8200 5750 50  0001 C CNN
-F 1 "+3V3" H 8215 6073 50  0000 C CNN
-F 2 "" H 8200 5900 50  0001 C CNN
-F 3 "" H 8200 5900 50  0001 C CNN
-	1    8200 5900
-	1    0    0    -1
-$EndComp
-Wire Wire Line
-	8200 5900 8200 5950
-Wire Wire Line
-	8200 5950 8650 5950
 Connection ~ 8200 5950
 Wire Wire Line
-	8650 6050 8600 6050
-Wire Wire Line
-	8600 6050 8600 6100
-Wire Wire Line
-	8650 5750 8350 5750
-Wire Wire Line
-	8350 5750 8350 5650
-Wire Wire Line
 	7850 5650 7850 5300
 Wire Wire Line
 	7850 5300 7500 5300
-Wire Wire Line
-	8650 5650 8400 5650
-Wire Wire Line
-	8400 5650 8400 5600
 $Comp
 L Device:C C15
@@
 Wire Wire Line
 	7900 5400 7500 5400
-Wire Wire Line
-	8400 5600 7900 5600
 Wire Wire Line
 	7900 5600 7900 5400
@@
 Wire Wire Line
 	2950 2250 2800 2250
+Wire Wire Line
+	8200 5900 8200 5950
+$Comp
+L power:+3V3 #PWR04
+U 1 1 610BDED3
+P 8200 5900
+F 0 "#PWR04" H 8200 5750 50  0001 C CNN
+F 1 "+3V3" H 8215 6073 50  0000 C CNN
+F 2 "" H 8200 5900 50  0001 C CNN
+F 3 "" H 8200 5900 50  0001 C CNN
+	1    8200 5900
+	1    0    0    -1
+$EndComp
+Wire Wire Line
+	9850 5150 9850 5950
+Wire Wire Line
+	9750 5250 9750 5750
+Wire Wire Line
+	8350 5750 8350 5650
+Wire Wire Line
+	8600 6050 8600 6100
+Wire Wire Line
+	8400 5600 7900 5600
+Wire Wire Line
+	8400 5650 8400 5600
+Wire Wire Line
+	8650 6050 8600 6050
+Wire Wire Line
+	9650 5750 9750 5750
+Wire Wire Line
+	9650 5950 9850 5950
+Wire Wire Line
+	8200 5950 8650 5950
+Wire Wire Line
+	8650 5750 8350 5750
+Wire Wire Line
+	9150 4950 9150 5450
+Wire Wire Line
+	9150 6300 9150 6250
+Wire Wire Line
+	8650 5650 8400 5650
+$Comp
+L Interface_CAN_LIN:MCP2558FD-xMF U5
+U 1 1 60F56096
+P 9150 5850
+F 0 "U5" H 9150 6431 50  0000 C CNN
+F 1 "TLE9250V" H 9150 6340 50  0000 C CNN
+F 2 "Package_SO:Infineon_PG-DSO-8-27_3.9x4.9mm_EP2.65x3mm" H 9150 5250 50  0001 C CNN
+F 3 "https://ww1.microchip.com/downloads/en/DeviceDoc/20005533A.pdf" H 9150 5850 50  0001 C CNN
+	1    9150 5850
+	1    0    0    -1
+$EndComp
+$Comp
+L power:GND #PWR0136
+U 1 1 610CB3DD
+P 7800 5950
+F 0 "#PWR0136" H 7800 5700 50  0001 C CNN
+F 1 "GND" H 7805 5777 50  0000 C CNN
+F 2 "" H 7800 5950 50  0001 C CNN
+F 3 "" H 7800 5950 50  0001 C CNN
+	1    7800 5950
+	0    1    1    0
+$EndComp
+Wire Wire Line
+	7800 5950 7850 5950
+$Comp
+L Device:C C10
+U 1 1 610A595F
+P 8000 5950
+F 0 "C10" H 8115 5996 50  0000 L CNN
+F 1 "100nF" H 8115 5905 50  0000 L CNN
+F 2 "Capacitor_SMD:C_0603_1608Metric" H 8038 5800 50  0001 C CNN
+F 3 "~" H 8000 5950 50  0001 C CNN
+	1    8000 5950
+	0    1    1    0
+$EndComp
+Wire Wire Line
+	10750 3650 10750 3850
+Connection ~ 10750 3650
 $EndSCHEMATC

Commit message: Make room for latching connector
Parts:
- J3: footprint Custom_FP:MicroMatch_04_Vertical_SMD -> Custom_FP:MicroMatch_04_Vertical_SMD_Lock
Changed lines of the file:
@@
 F 0 "J3" H 10530 5142 50  0000 L CNN
 F 1 "Conn_01x04" H 10530 5051 50  0000 L CNN
-F 2 "Custom_FP:MicroMatch_04_Vertical_SMD" H 10450 5150 50  0001 C CNN
+F 2 "Custom_FP:MicroMatch_04_Vertical_SMD_Lock" H 10450 5150 50  0001 C CNN
 F 3 "~" H 10450 5150 50  0001 C CNN
 	1    10450 5150
