File: CORE/MIDI_DIN.kicad_pcb (KiCad board)
At the start: 2 copper layers, 29.5 x 99.8 mm, 62 parts, among them J1 Conn_02x08_Odd_Even, J2 USB_C_Receptacle_USB2.0, J3 Conn_01x04, J5 MAB5100S, J6 MAB5100S, J7 Conn_01x06, Q1 BSS84, Q2 2N7002, Q5 2N7002, SW1 SW_Slide_SPDT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

Commit message: Fix DRC warnings
Parts:
- J5, J6: footprint Custom_FP:DIN-5_Hirschmann_MAB5100S -> Custom_FP:DIN-5_Hirschmann
Changed lines of the file:
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@@
     )
   )
-  (footprint "Custom_FP:DIN-5_Hirschmann_MAB5100S" (layer "F.Cu")
+  (footprint "Custom_FP:DIN-5_Hirschmann" (layer "F.Cu")
     (at 90 85.5)
     (property "Sheetfile" "MIDI_DIN.kicad_sch")
@@
         (effects (font (size 1 1) (thickness 0.15)))
     )
-    (fp_circle (center 0 0) (end 0 -7)
-      (stroke (width 0.12) (type solid)) (fill none) (layer "F.SilkS"))
+    (fp_arc (start 2.5 -7) (mid 0 7.1782) (end -2.5 -7)
+      (stroke (width 0.12) (type default)) (layer "F.SilkS"))
     (fp_circle (center 0 0) (end 0 10)
       (stroke (width 0.12) (type solid)) (fill none) (layer "F.SilkS"))
@@
       (net 23 "Net-(D6-A)") (pintype "passive"))
   )
-  (footprint "Custom_FP:DIN-5_Hirschmann_MAB5100S" (layer "F.Cu")
+  (footprint "Custom_FP:DIN-5_Hirschmann" (layer "F.Cu")
     (at 90 131.5)
     (property "Sheetfile" "MIDI_DIN.kicad_sch")
@@
         (effects (font (size 1 1) (thickness 0.15)))
     )
-    (fp_circle (center 0 0) (end 0 -7)
-      (stroke (width 0.12) (type solid)) (fill none) (layer "F.SilkS"))
+    (fp_arc (start 2.5 -7) (mid 0 7.1782) (end -2.5 -7)
+      (stroke (width 0.12) (type default)) (layer "F.SilkS"))
     (fp_circle (center 0 0) (end 0 10)
       (stroke (width 0.12) (type solid)) (fill none) (layer "F.SilkS"))
@@
     (property "ki_keywords" "CAN FD Controller SPI")
     (attr smd)
-    (fp_text reference "U4" (at 0 5.28) (layer "B.SilkS")
-        (effects (font (size 1 1) (thickness 0.15)) (justify mirror))
-    )
+    (fp_text reference "U4" (at -1.25 5.28) (layer "B.SilkS")
+        (effects (font (size 1 1) (thickness 0.15)) (justify mirror))
+    )

Commit message: Finalize module
Parts:
- C13, C14: value 15pF -> 12pF
- R18, R19: footprint Resistor_SMD:R_0603_1608Metric -> Resistor_SMD:R_0805_2012Metric
- moved C16 0.79 mm to (78.8, 50.5)
- moved R18 0.25 mm to (82.0, 49.5)
- moved R19 0.25 mm to (82.0, 51.5)
Other:
- rule pad_to_mask_clearance: 0.05 -> 0
